File: filscrete-8bp/filscrete-8bp.kicad_pcb (KiCad board)
At the start: 2 copper layers, 46.3 x 16 mm, 10 parts

Commit message: Added low noise LDO and USB plug footprint
A low noise LDO for use in sam has been added, together
with the footprint for a Molex USB A plug.
Changed lines of the file:
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@@
       (plot_on_all_layers_selection 0x0000000_00000000)
       (disableapertmacros false)
-      (usegerberextensions false)
-      (usegerberattributes true)
-      (usegerberadvancedattributes true)
-      (creategerberjobfile true)
+      (usegerberextensions true)
+      (usegerberattributes false)
+      (usegerberadvancedattributes false)
+      (creategerberjobfile false)
       (dashed_line_dash_ratio 12.000000)
       (dashed_line_gap_ratio 3.000000)
@@
       (psa4output false)
       (plotreference true)
-      (plotvalue true)
+      (plotvalue false)
       (plotinvisibletext false)
       (sketchpadsonfab false)
-      (subtractmaskfromsilk false)
+      (subtractmaskfromsilk true)
       (outputformat 1)
       (mirror false)
-      (drillshape 1)
+      (drillshape 0)
       (scaleselection 1)
-      (outputdirectory "")
+      (outputdirectory "/home/anton/Downloads/filscrete-8bp/")
     )
   )
@@
     (property "ki_keywords" "BNC SMA SMB SMC LEMO coaxial connector CINCH RCA")
     (attr smd)
-    (fp_text reference "OUT1" (at -4.5 -0.8 unlocked) (layer "F.SilkS")
+    (fp_text reference "OUT1" (at -4.5 -0.8 unlocked) (layer "F.SilkS") hide
         (effects (font (size 1.2 1.2) (thickness 0.1)))
     )
@@
     (property "ki_keywords" "BNC SMA SMB SMC LEMO coaxial connector CINCH RCA")
     (attr smd)
-    (fp_text reference "IN1" (at 4.5 -1.5 unlocked) (layer "F.SilkS")
+    (fp_text reference "IN1" (at 4.5 -1.5 unlocked) (layer "F.SilkS") hide
         (effects (font (size 1.2 1.2) (thickness 0.1)))
     )
