File: sam/sam.kicad_sch (KiCad schematic)
At the start: 4 parts, among them J1 USB_B_Micro, J2 Conn_Coaxial, U1 SPIRIT1, U2 STM32F070C6Tx

Commit message: Add 4 channel TVS diode array to lib
Parts:
- removed J1: USB_B_Micro, Connector_USB:USB_Micro-B_Molex_47346-0001, symbol Connector:USB_B_Micro
- added D1: DTS2042-04TS, Package_TO_SOT_SMD:TSOT-23-6, symbol pcrap:DTS2042-04TS
- added J1: USB_A, Connector_USB:USB_A_CONNFLY_DS1095-WNR0, symbol Connector:USB_A
Connections:
- net D+: now also D1.1, J1.2 (D-)
- net D-: now also D1.3, J1.3 (D+)
- net GND: now also D1.2, J1.4 (GND), J1.5 (Shield)
- new net 5V: D1.4, D1.6, J1.1 (VBUS)
Changed lines of the file:
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@@
 (kicad_sch (version 20230121) (generator eeschema)
   (paper "A4")
+  (junction (at 54.61 27.94) (diameter 0) (color 0 0 0 0)
+  )
+  (junction (at 41.91 36.83) (diameter 0) (color 0 0 0 0)
+  )
   (junction (at 109.22 118.11) (diameter 0) (color 0 0 0 0)
   )
   (junction (at 27.94 43.18) (diameter 0) (color 0 0 0 0)
   )
+  (junction (at 48.26 33.02) (diameter 0) (color 0 0 0 0)
+  )
+  (junction (at 60.96 27.94) (diameter 0) (color 0 0 0 0)
+  )
+  (wire (pts (xy 54.61 38.1) (xy 54.61 27.94))
+    (stroke (width 0) (type default))
+  )
+  (wire (pts (xy 54.61 27.94) (xy 38.1 27.94))
+    (stroke (width 0) (type default))
+  )
   (wire (pts (xy 27.94 43.18) (xy 30.48 43.18))
     (stroke (width 0) (type default))
@@
     (stroke (width 0) (type default))
   )
+  (wire (pts (xy 41.91 36.83) (xy 63.5 36.83))
+    (stroke (width 0) (type default))
+  )
+  (wire (pts (xy 60.96 27.94) (xy 60.96 38.1))
+    (stroke (width 0) (type default))
+  )
   (wire (pts (xy 212.09 93.98) (xy 219.71 93.98))
     (stroke (width 0) (type default))
@@
     (stroke (width 0) (type default))
   )
-  (wire (pts (xy 38.1 35.56) (xy 44.45 35.56))
+  (wire (pts (xy 41.91 36.83) (xy 41.91 35.56))
+    (stroke (width 0) (type default))
+  )
+  (wire (pts (xy 41.91 38.1) (xy 41.91 36.83))
+    (stroke (width 0) (type default))
+  )
+  (wire (pts (xy 38.1 35.56) (xy 41.91 35.56))
+    (stroke (width 0) (type default))
+  )
+  (wire (pts (xy 48.26 38.1) (xy 48.26 33.02))
+    (stroke (width 0) (type default))
+  )
+  (wire (pts (xy 60.96 27.94) (xy 54.61 27.94))
+    (stroke (width 0) (type default))
+  )
+  (wire (pts (xy 60.96 27.94) (xy 64.77 27.94))
+    (stroke (width 0) (type default))
+  )
+  (wire (pts (xy 38.1 33.02) (xy 48.26 33.02))
     (stroke (width 0) (type default))
   )
@@
   )
   (wire (pts (xy 105.41 118.11) (xy 109.22 118.11))
+    (stroke (width 0) (type default))
+  )
+  (wire (pts (xy 48.26 33.02) (xy 63.5 33.02))
     (stroke (width 0) (type default))
   )
@@
     )
   )
-  (global_label "D-" (shape input) (at 44.45 35.56 0) (fields_autoplaced)
-    (effects (font (size 1.27 1.27)) (justify left))
-    (property "Intersheetrefs" "${INTERSHEET_REFS}" (at 50.1982 35.56 0)
+  (global_label "D-" (shape input) (at 63.5 33.02 0) (fields_autoplaced)
+    (effects (font (size 1.27 1.27)) (justify left))
+    (property "Intersheetrefs" "${INTERSHEET_REFS}" (at 69.2482 33.02 0)
       (effects (font (size 1.27 1.27)) (justify left) hide)
     )
@@
     )
   )
+  (global_label "5V" (shape input) (at 64.77 27.94 0) (fields_autoplaced)
+    (effects (font (size 1.27 1.27)) (justify left))
+    (property "Intersheetrefs" "${INTERSHEET_REFS}" (at 69.9739 27.94 0)
+      (effects (font (size 1.27 1.27)) (justify left) hide)
+    )
+  )
   (global_label "CS" (shape input) (at 212.09 99.06 180) (fields_autoplaced)
     (effects (font (size 1.27 1.27)) (justify right))
@@
     )
   )
-  (global_label "D+" (shape input) (at 38.1 33.02 0) (fields_autoplaced)
-    (effects (font (size 1.27 1.27)) (justify left))
-    (property "Intersheetrefs" "${INTERSHEET_REFS}" (at 43.8482 33.02 0)
+  (global_label "D+" (shape input) (at 63.5 36.83 0) (fields_autoplaced)
+    (effects (font (size 1.27 1.27)) (justify left))
+    (property "Intersheetrefs" "${INTERSHEET_REFS}" (at 69.2482 36.83 0)
       (effects (font (size 1.27 1.27)) (justify left) hide)
     )
@@
     )
   )
-  (symbol (lib_id "power:GND") (at 109.22 118.11 0) (unit 1)
-    (in_bom yes) (on_board yes) (dnp no)
-    (property "Reference" "#PWR02" (at 109.22 124.46 0)
-      (effects (font (size 1.27 1.27)) hide)
-    )
-    (property "Value" "GND" (at 113.03 120.65 0)
-      (effects (font (size 1.27 1.27)))
-    )
-    (property "Footprint" "" (at 109.22 118.11 0)
-      (effects (font (size 1.27 1.27)) hide)
-    )
-    (property "Datasheet" "" (at 109.22 118.11 0)
-      (effects (font (size 1.27 1.27)) hide)
-    )
-    (pin "1")
-    (instances
-      (project "sam"
-        (path "/ebb33103-2b7d-42ff-9c11-2751d80bcdb8"
-          (reference "#PWR02") (unit 1)
-        )
-      )
-    )
-  )
-  (symbol (lib_id "Connector:USB_B_Micro") (at 30.48 33.02 0) (unit 1)
+  (symbol (lib_id "Connector:USB_A") (at 30.48 33.02 0) (unit 1)
     (in_bom yes) (on_board yes) (dnp no) (fields_autoplaced)
-    (property "Reference" "J1" (at 30.48 21.59 0)
-      (effects (font (size 1.27 1.27)))
-    )
-    (property "Value" "USB_B_Micro" (at 30.48 24.13 0)
-      (effects (font (size 1.27 1.27)))
-    )
-    (property "Footprint" "Connector_USB:USB_Micro-B_Molex_47346-0001" (at 34.29 34.29 0)
-      (effects (font (size 1.27 1.27)) hide)
-    )
-    (property "Datasheet" "~" (at 34.29 34.29 0)
+    (property "Reference" "J1" (at 30.48 20.32 0)
+      (effects (font (size 1.27 1.27)))
+    )
+    (property "Value" "USB_A" (at 30.48 22.86 0)
+      (effects (font (size 1.27 1.27)))
+    )
+    (property "Footprint" "Connector_USB:USB_A_CONNFLY_DS1095-WNR0" (at 34.29 34.29 0)
+      (effects (font (size 1.27 1.27)) hide)
+    )
+    (property "Datasheet" " ~" (at 34.29 34.29 0)
       (effects (font (size 1.27 1.27)) hide)
     )
@@
     (pin "4")
     (pin "5")
-    (pin "6")
     (instances
       (project "sam"
         (path "/ebb33103-2b7d-42ff-9c11-2751d80bcdb8"
           (reference "J1") (unit 1)
+        )
+      )
+    )
+  )
+  (symbol (lib_id "power:GND") (at 109.22 118.11 0) (unit 1)
+    (in_bom yes) (on_board yes) (dnp no)
+    (property "Reference" "#PWR02" (at 109.22 124.46 0)
+      (effects (font (size 1.27 1.27)) hide)
+    )
+    (property "Value" "GND" (at 113.03 120.65 0)
+      (effects (font (size 1.27 1.27)))
+    )
+    (property "Footprint" "" (at 109.22 118.11 0)
+      (effects (font (size 1.27 1.27)) hide)
+    )
+    (property "Datasheet" "" (at 109.22 118.11 0)
+      (effects (font (size 1.27 1.27)) hide)
+    )
+    (pin "1")
+    (instances
+      (project "sam"
+        (path "/ebb33103-2b7d-42ff-9c11-2751d80bcdb8"
+          (reference "#PWR02") (unit 1)
         )
       )
@@
     )
   )
+  (symbol (lib_id "pcrap:DTS2042-04TS") (at 50.8 36.83 0) (unit 1)
+    (in_bom yes) (on_board yes) (dnp no)
+    (property "Reference" "D1" (at 44.45 45.72 0)
+      (effects (font (size 1.27 1.27)) (justify right))
+    )
+    (property "Value" "DTS2042-04TS" (at 67.31 45.72 0)
+      (effects (font (size 1.27 1.27)) (justify right))
+    )
+    (property "Footprint" "Package_TO_SOT_SMD:TSOT-23-6" (at 50.8 26.67 0)
+      (effects (font (size 1.27 1.27)) hide)
+    )
+    (property "Datasheet" "https://www.diodes.com/assets/datasheets/DT2042-04TS.pdf" (at 50.8 29.21 0)
+      (effects (font (size 1.27 1.27)) hide)
+    )
+    (pin "1")
+    (pin "2")
+    (pin "3")
+    (pin "4")
+    (pin "5")
+    (pin "6")
+    (instances
+      (project "sam"
+        (path "/ebb33103-2b7d-42ff-9c11-2751d80bcdb8"
+          (reference "D1") (unit 1)
+        )
+      )
+    )
+  )
   (symbol (lib_id "pcrap:SPIRIT1") (at 92.71 102.87 0) (unit 1)
     (in_bom yes) (on_board yes) (dnp no) (fields_autoplaced)
@@
         )
       )
+    )
+  )
+  (symbol (lib_id "power:GND") (at 50.8 48.26 0) (unit 1)
+    (in_bom yes) (on_board yes) (dnp no) (fields_autoplaced)
+    (property "Reference" "#PWR07" (at 50.8 54.61 0)
+      (effects (font (size 1.27 1.27)) hide)
+    )
+    (property "Value" "GND" (at 50.8 53.34 0)
+      (effects (font (size 1.27 1.27)))
+    )
+    (property "Footprint" "" (at 50.8 48.26 0)
+      (effects (font (size 1.27 1.27)) hide)
+    )
+    (property "Datasheet" "" (at 50.8 48.26 0)
+      (effects (font (size 1.27 1.27)) hide)
+    )
+    (pin "1")
+    (instances
+      (project "sam"
+        (path "/ebb33103-2b7d-42ff-9c11-2751d80bcdb8"
+          (reference "#PWR07") (unit 1)
+        )
+      )

Commit message: Added low noise LDO and USB plug footprint
A low noise LDO for use in sam has been added, together
with the footprint for a Molex USB A plug.
Parts:
- added C1, C2: 1u, Capacitor_SMD:C_1206_3216Metric, symbol Device:C
- added C3: 100n, Capacitor_SMD:C_0805_2012Metric, symbol Device:C
- added C4, C5, C6: 100n, Capacitor_SMD:C_0603_1608Metric, symbol Device:C
- added FB1: FerriteBead, Inductor_SMD:L_0805_2012Metric, symbol Device:FerriteBead
- added R1: 100k, Resistor_SMD:R_0603_1608Metric, symbol Device:R
- added U2: LDLN030, Package_TO_SOT_SMD:TSOT-23-5, symbol pcrap:LDLN030
- J1: footprint Connector_USB:USB_A_CONNFLY_DS1095-WNR0 -> pcrap:USB_A_MOLEX_480372000
- renumbered U2 to U3
Connections:
- net 5V: now also C1.1, U2.1 (VIN), U2.3 (EN); no longer D1.6
- net D+: now also J1.3 (D+); no longer J1.2 (D-)
- net D-: now also J1.2 (D-); no longer J1.3 (D+)
- net GND: now also U3.23 (VSS), U3.35 (VSS), U3.47 (VSS), U3.8 (VSSA), C1.2, C2.2, C3.2, C4.2, C5.2, C6.2, U2.2 (GND)
- net 3V3: now reaches U3.1 (VDD)
- net 3V3: now also U3.24 (VDD), U3.36 (VDD), U3.48 (VDD), U3.9 (VDDA), C3.1, C4.1, C5.1, C6.1, FB1.2
- new net: R1.2, U2.4 (PG)
- new net LDO: C2.1, FB1.1, R1.1, U2.5 (OUT)
- no-connect marks 0 -> 1
