File: cocoro/cocoro.kicad_pcb (KiCad board)
At the start: 2 copper layers, 100 x 100 mm, 34 parts, among them J1 USB_B_Micro, J2 Conn_01x04_Pin, J3 Conn_01x04_Pin, Q1 FDN340P, Q2 FDN340P, Q3 FDN340P, U1 LED1642GWTTR

Commit message: cocoro: imp vbus protection, changed nets
Removed ESD and added two MLVs according to Littelfuse application
notes to protect the USB port from overvoltage. Changed nets for LEDs
to improve routing and moved the LED driver to what seems a better
position.

Added some extra components (rotary encoder among others) to the board.
Parts:
- removed the D1 at (180.0, 141.0)
- added C4: 100n, Capacitor_SMD:C_0805_2012Metric, F.Cu at (163.0, 143.0)
- added C5: 1u, Capacitor_SMD:C_1206_3216Metric, F.Cu at (150.3, 110.0)
- added RV2: V55MLA0603LNR, Resistor_SMD:R_0603_1608Metric, F.Cu at (177.0, 143.0)
- added SW1: SW_Push, Button_Switch_SMD:SW_Push_1P1T_NO_CK_KMR2, F.Cu at (134.5, 143.0)
- added SW2: RotaryEncoder_Switch, Rotary_Encoder:RotaryEncoder_Alps_EC11E-Switch_Vertical_H20mm, F.Cu at (104.0, 117.0)
- added U2: LED1642GWTTR, Package_SO:TSSOP-24_4.4x7.8mm_P0.65mm, F.Cu at (150.1, 116.6)
- C1: footprint Capacitor_SMD:C_0805_2012Metric -> Capacitor_SMD:C_0603_1608Metric
- C2: value 1u -> 100n
- C3: value 100n -> 1u; footprint Capacitor_SMD:C_0805_2012Metric -> Capacitor_SMD:C_1206_3216Metric
- FB1: value FerriteBead -> 220@100MHz
- U1: value LED1642GWTTR -> STM8S105K6; footprint Package_SO:TSSOP-24_4.4x7.8mm_P0.65mm -> Package_QFP:LQFP-32_7x7mm_P0.8mm
- moved C1 35.0 mm to (131.0, 142.8), turned to 90 degrees
- moved U1 26.7 mm to (124.8, 135.0), turned to 180 degrees
- moved C2 11.7 mm to (173.0, 140.0)
- moved C3 7.07 mm to (166.0, 143.0)
- moved F1 6.71 mm to (178.0, 137.0), turned to 90 degrees
- moved RV1 6.40 mm to (184.0, 143.0), turned to 180 degrees
- moved FB1 5.39 mm to (169.0, 139.0)
- moved J2 4.27 mm to (124.0, 145.5)
- renumbered D2 to D1, D11 to D10, D12 to D11, D13 to D12, D14 to D13, D15 to D14, D16 to D15, D17 to D16, D3 to D2, D4 to D3, D5 to D4, D6 to D5, D7 to D6, D8 to D7, D9 to D8, D10 to D9
Connections:
- C1 pad 1: /FUSED_VBUS -> GND
- C1 pad 2: GND -> RST
- C2 pad 1: 5V -> /FUSED_VBUS
- D10 pad 2: OUT9 -> OUT7
- D11 pad 2: OUT10 -> OUT6
- D12 pad 2: OUT11 -> OUT5
- D13 pad 2: OUT12 -> OUT4
- D14 pad 2: OUT13 -> OUT3
- D15 pad 2: OUT14 -> OUT2
- D16 pad 2: OUT15 -> OUT1
- D2 pad 2: OUT1 -> OUT15
- D3 pad 2: OUT2 -> OUT14
- D4 pad 2: OUT3 -> OUT13
- D5 pad 2: OUT4 -> OUT12
- D6 pad 2: OUT5 -> OUT11
- D7 pad 2: OUT6 -> OUT10
- D8 pad 2: OUT7 -> OUT9
- J1 pad 6: GND -> SHLD
- J2 pad 2: SWIM -> GND
- J2 pad 3: GND -> SWIM
- J3 pad 2: VDD -> 5V
- RV1 pad 1: /VBUS -> SHLD
- U1 pad 1: GND -> RST
- U1 pad 10: OUT5 -> unconnected-(U1-VSSA-Pad10)
- U1 pad 11: OUT6 -> SDA
- U1 pad 12: OUT7 -> SCL
- U1 pad 13: OUT8 -> unconnected-(U1-PB3-Pad13)
- U1 pad 14: OUT9 -> EN_BLUE
- U1 pad 15: OUT10 -> EN_GREEN
- U1 pad 16: OUT11 -> EN_RED
- U1 pad 17: OUT12 -> unconnected-(U1-PE5-Pad17)
- U1 pad 18: OUT13 -> unconnected-(U1-PC1-Pad18)
- U1 pad 19: OUT14 -> unconnected-(U1-PC2-Pad19)
- U1 pad 20: OUT15 -> unconnected-(U1-PC3-Pad20)
- U1 pad 5: OUT0 -> unconnected-(U1-VCAP-Pad5)
- U1 pad 6: OUT1 -> unconnected-(U1-VDD-Pad6)
- U1 pad 7: OUT2 -> unconnected-(U1-VDDIO-Pad7)
- U1 pad 8: OUT3 -> unconnected-(U1-PF4-Pad8)
- U1 pad 9: OUT4 -> unconnected-(U1-VDDA-Pad9)
Other:
- board text added: "0.0.1v"
- board text added: "COCORO"
- board text added: "RESET"
- board text added: "VDD GND SWIM RST"

Commit message: cocoro: Finish MCU and LED driver section
Passive components were added to the MCU and the connections
to the led driver were drawn to the schematic. Remaining free
pins have been connected to headers for external use.
Parts:
- added C6: 1u, Capacitor_SMD:C_1206_3216Metric, F.Cu at (139.7, 135.0)
- added C7: 100n, Capacitor_SMD:C_0603_1608Metric, F.Cu at (134.2, 128.0)
- added C8: 100n, Capacitor_SMD:C_0603_1608Metric, F.Cu at (138.2, 131.0)
- moved SW1 6.63 mm to (141.1, 143.2), turned to 180 degrees
- moved J2 6.18 mm to (130.2, 145.5)
- moved U1 6.17 mm to (131.0, 135.0)
- moved C1 5.23 mm to (136.2, 142.0)
- moved J3 3.00 mm to (148.5, 93.0)
- moved C2 2.00 mm to (171.0, 140.0)
- moved C3 2.00 mm to (164.0, 143.0)
- moved C4 2.00 mm to (161.0, 143.0)
- moved F1 2.00 mm to (176.0, 137.0)
- moved FB1 2.00 mm to (167.0, 139.0)
- moved J1 2.00 mm to (178.0, 147.2)
- moved RV1 2.00 mm to (182.0, 143.0)
- moved RV2 2.00 mm to (175.0, 143.0)
Connections:
- U1 pad 10: unconnected-(U1-VSSA-Pad10) -> GND
- U1 pad 17: unconnected-(U1-PE5-Pad17) -> CLICK
- U1 pad 18: unconnected-(U1-PC1-Pad18) -> ENC_A
- U1 pad 19: unconnected-(U1-PC2-Pad19) -> ENC_B
- U1 pad 4: unconnected-(U1-VSS-Pad4) -> GND
- U1 pad 5: unconnected-(U1-VCAP-Pad5) -> Net-(U1-VCAP)
- U1 pad 6: unconnected-(U1-VDD-Pad6) -> 5V
- U1 pad 7: unconnected-(U1-VDDIO-Pad7) -> 5V
- U1 pad 9: unconnected-(U1-VDDA-Pad9) -> 5V

Commit message: cocoro: Route board
The board has been completely routed. Still needs a double check.
The LED footprint has been changed to something that has more
space between pins, in order to make it easier to manufacture.
Parts:
- added C1: 100n, Capacitor_SMD:C_0603_1608Metric, F.Cu at (189.5, 125.7)
- added J4: Conn_01x10_Pin, Connector_PinHeader_2.54mm:PinHeader_1x10_P2.54mm_Vertical, F.Cu at (103.0, 138.0)
- added R1: 5.1k, Resistor_SMD:R_0603_1608Metric, F.Cu at (187.5, 134.7)
- added R2: 11k, Resistor_SMD:R_0603_1608Metric, F.Cu at (156.0, 112.0)
- added U1: DHT11, Sensor:Aosong_DHT11_5.5x12.0_P2.54mm, F.Cu at (185.9, 130.0)
- D1, D10, D11, D12, D13, D14, D15, D16, D2, D3, D4, D5, D6, D7, D8, D9: footprint LED_THT:LED_D5.0mm-4_RGB -> LED_THT:LED_D5.0mm-4_RGB_Staggered_Pins
- J2, J3: footprint Connector_PinHeader_1.00mm:PinHeader_1x04_P1.00mm_Vertical -> Connector_PinHeader_2.54mm:PinHeader_1x04_P2.54mm_Vertical
- moved J2 6.26 mm to (123.9, 145.5)
- moved SW1 5.39 mm to (109.0, 119.0)
- moved C4 3.50 mm to (136.2, 145.5)
- moved J3 2.62 mm to (145.9, 93.0)
- moved SW2 2.05 mm to (141.2, 145.2)
- moved C8 1.56 mm to (138.5, 136.0), turned to -90 degrees
- moved RV2 1.00 mm to (174.0, 143.0)
- moved C6 0.57 mm to (134.8, 128.0)
- moved C5 0.50 mm to (161.0, 142.5)
- moved C7 0.07 mm to (138.2, 131.0)
- renumbered C1 to C4, C4 to C5, C7 to C6, C8 to C7, C6 to C8, C5 to C9, SW2 to SW1, SW1 to SW2, U1 to U2, U2 to U3
Connections:
- J2 pad 1: VDD -> 5V
- U2 pad 13: unconnected-(U1-PB3-Pad13) -> EN_BLUE
- U2 pad 14: EN_BLUE -> EN_GREEN
- U2 pad 15: EN_GREEN -> EN_RED
- U2 pad 16: EN_RED -> ADC0
- U2 pad 20: unconnected-(U1-PC3-Pad20) -> /PC3
- U2 pad 21: unconnected-(U1-PC4-Pad21) -> /PC4
- U2 pad 22: unconnected-(U1-PC5-Pad22) -> /PC5
- U2 pad 23: unconnected-(U1-PC7-Pad23) -> /PC6
- U2 pad 24: unconnected-(U1-PC7-Pad24) -> /PC7
- U2 pad 25: unconnected-(U1-PD0-Pad25) -> /PD0
- U2 pad 27: unconnected-(U1-PD2-Pad27) -> PWCLK
- U2 pad 28: unconnected-(U1-PD3-Pad28) -> MISO
- U2 pad 29: unconnected-(U1-PD4-Pad29) -> MOSI
- U2 pad 30: unconnected-(U1-PD5-Pad30) -> SCLK
- U2 pad 31: unconnected-(U1-PD6-Pad31) -> LE
- U2 pad 32: unconnected-(U1-PD7-Pad32) -> DHT22
- U2 pad 8: unconnected-(U1-PF4-Pad8) -> ADC1
- U3 pad 2: unconnected-(U2-SDI-Pad2) -> MOSI
- U3 pad 21: unconnected-(U2-PWCLK-Pad21) -> PWCLK
- U3 pad 22: unconnected-(U2-SDO-Pad22) -> MISO
- U3 pad 23: unconnected-(U2-R-EXT-Pad23) -> /ledc/REXT
- U3 pad 3: unconnected-(U2-CLK-Pad3) -> SCLK
- U3 pad 4: unconnected-(U2-LE-Pad4) -> LE
Routing:
- net RED: track 0.00 -> 282.9 mm
- net GREEN: track 0.00 -> 276.1 mm, vias 0 -> 1
- net BLUE: track 0.00 -> 271.8 mm
- net DHT22: track 0.00 -> 69.7 mm, vias 0 -> 1
- net OUT2: track 0.00 -> 69.2 mm, vias 0 -> 1
- net OUT14: track 0.00 -> 69.2 mm
- net OUT3: track 0.00 -> 63.4 mm, vias 0 -> 1
- net OUT13: track 0.00 -> 63.2 mm
- net OUT4: track 0.00 -> 59.5 mm, vias 0 -> 1
- net EN_BLUE: track 0.00 -> 59.1 mm
- net OUT15: track 0.00 -> 56.1 mm
- net OUT1: track 0.00 -> 56.0 mm, vias 0 -> 1
- net EN_GREEN: track 0.00 -> 54.0 mm
- net OUT12: track 0.00 -> 52.4 mm
- net EN_RED: track 0.00 -> 50.7 mm
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- added copper zone on F.Cu, net 5V
- added copper zone on In2.Cu, net 5V
- added copper zone on B.Cu, net GND
- added copper zone on F.Cu, net GND
- added copper zone on In1.Cu, net GND
- added copper zone on F.Cu, net SHLD
Other:
- copper layers 2 -> 4
- board text added: "CORAÇÃO"
- board text added: "GND"
- board text added: "PB0"
- board text added: "PC3"
- board text added: "PC4"
- board text added: "PC5"
- board text added: "PC6"
- board text added: "PC7"
- board text added: "PD0"
- board text added: "PF4"
- board text added: "VDD"
- board text removed: "COCORO"

Commit message: cocoro: Board touchups and decoupling caps
Performed minor touchup to reduce the size of ground islands. Added
some extra vias and decoupling caps for the power MOSFETs, since
it is recommended to add some extra capacitance to the voltage line
according to the LED1642 datasheet.
Parts:
- added C10: TBD, Capacitor_SMD:C_0805_2012Metric, F.Cu at (159.2, 89.8)
- added C11: TBD, Capacitor_SMD:C_0805_2012Metric, F.Cu at (150.8, 89.0)
- added C12: TBD, Capacitor_SMD:C_0805_2012Metric, F.Cu at (145.2, 81.0)
- moved SW2 0.56 mm to (141.0, 145.8)
Routing:
- net 5V: track 28.8 -> 42.5 mm
- net GND: track 39.6 -> 32.3 mm, vias 30 -> 40
- net OUT14: track 69.2 -> 73.7 mm
- net OUT2: track 69.2 -> 73.4 mm
- net OUT4: track 59.5 -> 56.0 mm
- net RED: track 282.9 -> 286.1 mm
- net GREEN: track 276.1 -> 277.6 mm
- net PWCLK: track 47.7 -> 48.9 mm
- net EN_GREEN: track 54.0 -> 53.0 mm
- net EN_BLUE: track 59.1 -> 59.8 mm

Commit message: cocoro: Improve manufacturability and better placement
Vias on the left side of the LED1642 were far too close to be
easily manufactured by JLCPCB. Routing has been changed
to add more clearance to said vias.

The CORACAO text and version were moved to a better location to
ensure they are not covered by the DHT22 sensor.

Traces on LEDs were changed to 4mm to increase clearance between
traces and THT holes.

Traces for the MCU have all been set to 3mm to increase clearance
as well.

PCB corners have been rounded.

The switching MOSFETs and the LED above them were moved up
to give more space for the 0.96' display and ensure it does
not cover any LEDs.
Parts:
- moved C10 15.6 mm to (144.5, 84.8), turned to 180 degrees
- moved C11 7.98 mm to (157.5, 84.8)
- moved C12 6.89 mm to (151.0, 84.8), turned to 180 degrees
- moved Q3 4.60 mm to (157.0, 81.5)
- moved Q2 4.53 mm to (150.5, 81.5)
- moved Q1 4.50 mm to (144.0, 81.5)
- moved J3 3.91 mm to (147.0, 89.2)
- moved R1 0.99 mm to (188.5, 134.8), turned to 90 degrees
- moved D1 0.75 mm to (148.0, 74.2)
- moved C6 0.50 mm to (134.8, 127.5)
Routing:
- net RED: track 286.1 -> 275.7 mm
- net OUT0: track 46.6 -> 54.4 mm
- net SDA: track 46.6 -> 52.2 mm
- net EN_GREEN: track 53.0 -> 58.4 mm
- net GREEN: track 277.6 -> 272.8 mm
- net DHT22: track 69.7 -> 65.1 mm
- net SCL: track 45.9 -> 50.1 mm
- net EN_RED: track 50.7 -> 54.7 mm
- net EN_BLUE: track 59.8 -> 63.8 mm
- net OUT4: track 56.0 -> 53.1 mm
- net OUT5: track 41.1 -> 38.5 mm
- net GND: track 32.3 -> 30.4 mm, vias 40 -> 43
- net OUT6: track 32.1 -> 30.5 mm
- net BLUE: track 271.8 -> 270.5 mm
- net 5V: track 42.5 -> 42.2 mm, vias 12 -> 13
Other:
- outline, holes or cut-outs redrawn
- board text added: "I2C SCREEN"
- board text added: "JLCJLCJLCJLC"
- board text added: "github.com/crazybolillo/pcrap/cocoro"

Commit message: cocoro: fix footprints
* A new USB footprint for the actual product in hand has been added.
* The footprint for the RESET button was corrected to the actual
product in hand.
* Vias under the MCU were moved a little bit more to the center
for increased clearance from pads.
Parts:
- J1: footprint Connector_USB:USB_Micro-B_Molex_47346-0001 -> pcrap:USB_Micro-B_SHOU_HAN_MICRO_XNJ_ZB
- SW2: footprint Button_Switch_SMD:SW_Push_1P1T_NO_CK_KMR2 -> Button_Switch_SMD:SW_SPST_PTS810
- moved J1 5.05 mm to (178.1, 142.2), turned to 180 degrees
- moved RV1 0.50 mm to (182.0, 142.5)
- moved RV2 0.50 mm to (174.0, 142.5)
- moved SW2 0.50 mm to (141.5, 145.8)
Routing:
- net SHLD: track 0.00 -> 9.07 mm
- net GND: track 30.4 -> 29.5 mm, vias 43 -> 42
- net ADC1: track 37.0 -> 37.6 mm
- net /VBUS: track 7.81 -> 8.36 mm
