File: cocoro/cocoro.kicad_sch (KiCad schematic)
At the start: 14 parts, among them J1 USB_B_Micro, J2 Conn_01x04_Pin, J3 Conn_01x04_Pin

Commit message: cocoro: imp vbus protection, changed nets
Removed ESD and added two MLVs according to Littelfuse application
notes to protect the USB port from overvoltage. Changed nets for LEDs
to improve routing and moved the LED driver to what seems a better
position.

Added some extra components (rotary encoder among others) to the board.
Parts:
- removed D1: TPD1E10B06DYAR, Diode_SMD:D_SOD-523, symbol Device:D_Zener
- added C1: 100n, Capacitor_SMD:C_0603_1608Metric, symbol Device:C
- added RV1: V55MLA0603LNR, Resistor_SMD:R_0603_1608Metric, symbol Device:Varistor
- added SW1: SW_Push, Button_Switch_SMD:SW_Push_1P1T_NO_CK_KMR2, symbol Switch:SW_Push
- added SW2: RotaryEncoder_Switch, Rotary_Encoder:RotaryEncoder_Alps_EC11E-Switch_Vertical_H20mm, symbol Device:RotaryEncoder_Switch
- added U1: STM8S105K6, Package_QFP:LQFP-32_7x7mm_P0.8mm, symbol pcrap:STM8S105K6
- C3: renamed from C2; footprint Capacitor_SMD:C_0805_2012Metric -> Capacitor_SMD:C_1206_3216Metric
- FB1: value FerriteBead -> 220@100MHz
- renumbered C1 to C2, C3 to C4, RV1 to RV2
Connections:
- net GND: now also J2.2 (Pin_2), C1.1, RV1.2, SW1.1, SW2.C, SW2.S2; no longer J1.6 (Shield), J2.3 (Pin_3), RV2.2
- net RST: now also C1.2, SW1.2, U1.1 (~{RST})
- net SCL: now also U1.12 (PB4)
- net SDA: now also U1.11 (PB5)
- net SWIM: now also J2.3 (Pin_3), U1.26 (PD1); no longer J2.2 (Pin_2)
- new net CLICK: SW2.S1
- new net ENC_A: SW2.A
- new net ENC_B: SW2.B
- new net EN_BLUE: U1.14 (PB2)
- new net EN_GREEN: U1.15 (PB1)
- new net EN_RED: U1.16 (PB0)
- new net SHLD: J1.6 (Shield), RV1.1, RV2.2
- no-connect marks 3 -> 5
Other:
- note added: "MAIN MCU"
- moved on the sheet: C2, C3, C4, F1, FB1, J1, J2, J3, RV2

Commit message: cocoro: Finish MCU and LED driver section
Passive components were added to the MCU and the connections
to the led driver were drawn to the schematic. Remaining free
pins have been connected to headers for external use.
Parts:
- added C6: 1u, Capacitor_SMD:C_1206_3216Metric, symbol Device:C
- added C7, C8: 100n, Capacitor_SMD:C_0603_1608Metric, symbol Device:C
- added J4: Conn_01x08_Pin, Connector_PinHeader_1.00mm:PinHeader_1x08_P1.00mm_Vertical, symbol Connector:Conn_01x08_Pin
Connections:
- net 5V: now also U1.6 (VDD), U1.7 (VDDIO), U1.9 (VDDA), C7.1, C8.1
- net CLICK: now also U1.17 (PE5)
- net ENC_A: now also U1.18 (PC1)
- net ENC_B: now also U1.19 (PC2)
- net EN_BLUE: now also U1.13 (PB3); no longer U1.14 (PB2)
- net EN_GREEN: now also U1.14 (PB2); no longer U1.15 (PB1)
- net EN_RED: now also U1.15 (PB1); no longer U1.16 (PB0)
- net GND: now also U1.10 (VSSA), U1.4 (VSS), C6.2, C7.2, C8.2
- net at U1.20 (PC3): now also J4.6 (Pin_6)
- net at U1.21 (PC4): now also J4.5 (Pin_5)
- net at U1.22 (PC5): now also J4.4 (Pin_4)
- net at U1.23 (PC7): now also J4.3 (Pin_3)
- net at U1.24 (PC7): now also J4.2 (Pin_2)
- net at U1.25 (PD0): now also J4.1 (Pin_1)
- net DHT22: now reaches U1.27 (PD2)
- net MISO: now reaches U1.28 (PD3)
- net MOSI: now reaches U1.29 (PD4)
- net SCLK: now reaches U1.30 (PD5)
- net LE: now reaches U1.31 (PD6)
- net PWCLK: now reaches U1.32 (PD7)
- net at U1.5 (VCAP): now also C6.1
- net ADC0: now reaches U1.8 (PF4)
- net ADC0: now also J4.7 (Pin_7)
- new net ADC1: J4.8 (Pin_8), U1.16 (PB0)
Other:
- note added: "RESET CIRCUITRY"
- note added: "ROTARY ENCODER"
- moved on the sheet: C1, SW1, SW2, U1

Commit message: cocoro: Route board
The board has been completely routed. Still needs a double check.
The LED footprint has been changed to something that has more
space between pins, in order to make it easier to manufacture.
Parts:
- added C1: 100n, Capacitor_SMD:C_0603_1608Metric, symbol Device:C
- added R1: 5.1k, Resistor_SMD:R_0603_1608Metric, symbol Device:R
- added U1: DHT11, Sensor:Aosong_DHT11_5.5x12.0_P2.54mm, symbol Sensor:DHT11
- J2, J3: footprint Connector_PinHeader_1.00mm:PinHeader_1x04_P1.00mm_Vertical -> Connector_PinHeader_2.54mm:PinHeader_1x04_P2.54mm_Vertical
- J4: value Conn_01x08_Pin -> Conn_01x10_Pin; footprint Connector_PinHeader_1.00mm:PinHeader_1x08_P1.00mm_Vertical -> Connector_PinHeader_2.54mm:PinHeader_1x10_P2.54mm_Vertical; symbol Connector:Conn_01x08_Pin -> Connector:Conn_01x10_Pin
- renumbered C1 to C4, C4 to C5, C7 to C6, C8 to C7, C6 to C8, SW2 to SW1, SW1 to SW2, U1 to U2
Connections:
- net VDD is gone; now on net 5V: J2.1 (Pin_1)
- net 5V: now also J4.10 (Pin_10), C1.1, R1.1, U1.1 (VCC)
- net ADC0: now also J4.8 (Pin_8), U2.16 (PB0); no longer J4.7 (Pin_7), U2.8 (PF4)
- net ADC1: now also J4.7 (Pin_7), U2.8 (PF4); no longer J4.8 (Pin_8), U2.16 (PB0)
- net DHT22: now also U2.32 (PD7), R1.2, U1.2 (IO); no longer U2.27 (PD2)
- net GND: now also J4.9 (Pin_9), C1.2, U1.4 (GND)
- net PWCLK: now also U2.27 (PD2); no longer U2.32 (PD7)
- net PC3: now reaches J4.6 (Pin_6), U2.20 (PC3)
- net PC4: now reaches J4.5 (Pin_5), U2.21 (PC4)
- net PC5: now reaches J4.4 (Pin_4), U2.22 (PC5)
- net PC6: now reaches J4.3 (Pin_3), U2.23 (PC6)
- net PC7: now reaches J4.2 (Pin_2), U2.24 (PC7)
- net PD0: now reaches J4.1 (Pin_1), U2.25 (PD0)
Other:
- note added: "DHT11/22 SENSOR"

Commit message: cocoro: fix footprints
* A new USB footprint for the actual product in hand has been added.
* The footprint for the RESET button was corrected to the actual
product in hand.
* Vias under the MCU were moved a little bit more to the center
for increased clearance from pads.
Parts:
- J1: footprint Connector_USB:USB_Micro-B_Molex_47346-0001 -> pcrap:USB_Micro-B_SHOU_HAN_MICRO_XNJ_ZB
- SW2: footprint Button_Switch_SMD:SW_Push_1P1T_NO_CK_KMR2 -> Button_Switch_SMD:SW_SPST_PTS810
Changed lines of the file:
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@@
       (effects (font (size 1.27 1.27)))
     )
-    (property "Footprint" "Connector_USB:USB_Micro-B_Molex_47346-0001" (at 29.21 33.02 0)
+    (property "Footprint" "pcrap:USB_Micro-B_SHOU_HAN_MICRO_XNJ_ZB" (at 29.21 33.02 0)
       (effects (font (size 1.27 1.27)) hide)
     )
@@
       (effects (font (size 1.27 1.27)))
     )
-    (property "Footprint" "Button_Switch_SMD:SW_Push_1P1T_NO_CK_KMR2" (at 95.25 106.68 0)
-      (effects (font (size 1.27 1.27)) hide)
-    )
+    (property "Footprint" "Button_Switch_SMD:SW_SPST_PTS810" (at 95.25 106.68 0)
+      (effects (font (size 1.27 1.27)) hide)
+    )

Commit message: Housekeeping, deleted extra-crappy projects, add CI
Deleted a bunch of half-finished projects that won't be getting
attention anytime soon:

* filscrete-8bp: Making a good quality filter for the VHF band will be
  much harder than expected and won't be pursued for the time being.
* ev1496: Much more investigation needs to be done on the intrinsic
  characteristics of the MC1496 IC before being able to develop an
  evaluation board.
* sam: Very ambitious project, will start first with smaller ones.

Library symbols for these projects have been kept since they mave prove
useful in the future.

Front matter has been added to the remaining project. It is planned to
automatically create a portfolio website for this repo with balba:

https://gitlab.com/zoftko/balba

And a standard front matter will be needed for that.

Finally, a basic CI with pre-commit has been added to improve code
quality. In the future it should also perform spell checks.
Other:
- title: (none) -> User interface for controlling RGB LED Array
Changed lines of the file:
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@@
 (kicad_sch (version 20230121) (generator eeschema)
   (paper "A4")
+  (title_block
+    (title "User interface for controlling RGB LED Array")
+  )
   (junction (at 175.26 124.46) (diameter 0) (color 0 0 0 0)
   )
