File: cocoro/ledc.kicad_sch (KiCad schematic)
At the start: 20 parts, among them Q1 FDN340P, Q2 FDN340P, Q3 FDN340P, U1 LED1642GWTTR

Commit message: cocoro: imp vbus protection, changed nets
Removed ESD and added two MLVs according to Littelfuse application
notes to protect the USB port from overvoltage. Changed nets for LEDs
to improve routing and moved the LED driver to what seems a better
position.

Added some extra components (rotary encoder among others) to the board.
Parts:
- added C5: 1u, Capacitor_SMD:C_1206_3216Metric, symbol Device:C
Connections:
- net 5V: now also U1.24 (VDD), C5.1
- net GND: now also C5.2
- net OUT1: now also D17.2 (K); no longer D3.2 (K)
- net OUT10: now also D8.2 (K); no longer D12.2 (K)
- net OUT11: now also D7.2 (K); no longer D13.2 (K)
- net OUT12: now also D6.2 (K); no longer D14.2 (K)
- net OUT13: now also D5.2 (K); no longer D15.2 (K)
- net OUT14: now also D4.2 (K); no longer D16.2 (K)
- net OUT15: now also D3.2 (K); no longer D17.2 (K)
- net OUT2: now also D16.2 (K); no longer D4.2 (K)
- net OUT3: now also D15.2 (K); no longer D5.2 (K)
- net OUT4: now also D14.2 (K); no longer D6.2 (K)
- net OUT5: now also D13.2 (K); no longer D7.2 (K)
- net OUT6: now also D12.2 (K); no longer D8.2 (K)
- net OUT7: now also D11.2 (K); no longer D9.2 (K)
- net OUT9: now also D9.2 (K); no longer D11.2 (K)

Commit message: cocoro: Finish MCU and LED driver section
Passive components were added to the MCU and the connections
to the led driver were drawn to the schematic. Remaining free
pins have been connected to headers for external use.
Connections:
- net MOSI: now reaches U1.2 (SDI)
- net PWCLK: now reaches U1.21 (PWCLK)
- net MISO: now reaches U1.22 (SDO)
- net SCLK: now reaches U1.3 (CLK)
- net LE: now reaches U1.4 (LE)
Changed lines of the file:
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@@
   (junction (at 200.66 29.21) (diameter 0) (color 0 0 0 0)
   )
+  (wire (pts (xy 50.8 44.45) (xy 60.96 44.45))
+    (stroke (width 0) (type default))
+  )
   (wire (pts (xy 91.44 74.93) (xy 100.33 74.93))
     (stroke (width 0) (type default))
@@
     (stroke (width 0) (type default))
   )
+  (wire (pts (xy 59.69 54.61) (xy 60.96 54.61))
+    (stroke (width 0) (type default))
+  )
+  (wire (pts (xy 59.69 46.99) (xy 60.96 46.99))
+    (stroke (width 0) (type default))
+  )
   (wire (pts (xy 91.44 59.69) (xy 100.33 59.69))
     (stroke (width 0) (type default))
@@
     (stroke (width 0) (type default))
   )
+  (wire (pts (xy 50.8 49.53) (xy 60.96 49.53))
+    (stroke (width 0) (type default))
+  )
   (wire (pts (xy 227.33 82.55) (xy 223.52 82.55))
     (stroke (width 0) (type default))
@@
   )
   (wire (pts (xy 21.59 45.72) (xy 21.59 48.26))
+    (stroke (width 0) (type default))
+  )
+  (wire (pts (xy 59.69 41.91) (xy 60.96 41.91))
     (stroke (width 0) (type default))
   )
@@
     )
   )
+  (global_label "SCLK" (shape input) (at 59.69 46.99 180) (fields_autoplaced)
+    (effects (font (size 1.27 1.27)) (justify right))
+    (property "Intersheetrefs" "${INTERSHEET_REFS}" (at 52.0066 46.99 0)
+      (effects (font (size 1.27 1.27)) (justify right) hide)
+    )
+  )
+  (global_label "PWCLK" (shape input) (at 59.69 54.61 180) (fields_autoplaced)
+    (effects (font (size 1.27 1.27)) (justify right))
+    (property "Intersheetrefs" "${INTERSHEET_REFS}" (at 50.4947 54.61 0)
+      (effects (font (size 1.27 1.27)) (justify right) hide)
+    )
+  )
   (global_label "BLUE" (shape input) (at 227.33 133.35 180) (fields_autoplaced)
     (effects (font (size 1.27 1.27)) (justify right))
@@
     )
   )
+  (global_label "LE" (shape input) (at 50.8 49.53 180) (fields_autoplaced)
+    (effects (font (size 1.27 1.27)) (justify right))
+    (property "Intersheetrefs" "${INTERSHEET_REFS}" (at 45.7171 49.53 0)
+      (effects (font (size 1.27 1.27)) (justify right) hide)
+    )
+  )
+  (global_label "MISO" (shape input) (at 59.69 41.91 180) (fields_autoplaced)
+    (effects (font (size 1.27 1.27)) (justify right))
+    (property "Intersheetrefs" "${INTERSHEET_REFS}" (at 52.188 41.91 0)
+      (effects (font (size 1.27 1.27)) (justify right) hide)
+    )
+  )
   (global_label "BLUE" (shape input) (at 227.33 110.49 180) (fields_autoplaced)
     (effects (font (size 1.27 1.27)) (justify right))
@@
       (effects (font (size 1.27 1.27)) (justify right) hide)
     )
+  )
+  (global_label "MOSI" (shape input) (at 50.8 44.45 180) (fields_autoplaced)
+    (effects (font (size 1.27 1.27)) (justify right))
+    (property "Intersheetrefs" "${INTERSHEET_REFS}" (at 43.298 44.45 0)
+      (effects (font (size 1.27 1.27)) (justify right) hide)
+    )

Commit message: cocoro: Route board
The board has been completely routed. Still needs a double check.
The LED footprint has been changed to something that has more
space between pins, in order to make it easier to manufacture.
Parts:
- added R2: 11k, Resistor_SMD:R_0603_1608Metric, symbol Device:R
- D10, D11, D12, D13, D14, D15, D16, D17, D2, D3, D4, D5, D6, D7, D8, D9: footprint LED_THT:LED_D5.0mm-4_RGB -> LED_THT:LED_D5.0mm-4_RGB_Staggered_Pins
- renumbered C5 to C9
Connections:
- net GND: now also R2.2
- net REXT: now reaches U1.23 (R-EXT)
- net REXT: now also R2.1
Changed lines of the file:
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@@
+    (stroke (width 0) (type default))
+  )
+  (wire (pts (xy 55.88 68.58) (xy 55.88 67.31))
     (stroke (width 0) (type default))
   )
@@
     (stroke (width 0) (type default))
   )
+  (wire (pts (xy 55.88 67.31) (xy 60.96 67.31))
+    (stroke (width 0) (type default))
+  )
   (wire (pts (xy 91.44 64.77) (xy 100.33 64.77))
     (stroke (width 0) (type default))
@@
     (effects (font (size 2.54 2.54)) (justify left bottom))
   )
+  (label "REXT" (at 55.88 67.31 0) (fields_autoplaced)
+    (effects (font (size 1.27 1.27)) (justify left bottom))
+  )
   (global_label "BLUE" (shape input) (at 227.33 87.63 180) (fields_autoplaced)
     (effects (font (size 1.27 1.27)) (justify right))
@@
         )
         (path "/d9dd42f0-aa5c-442e-a67c-269b1cf4745b/97ea76ca-9415-4083-9485-343aeb93230e"
-          (reference "#PWR09") (unit 1)
+          (reference "#PWR012") (unit 1)
         )
       )
@@
       (effects (font (size 1.27 1.27)))
     )
-    (property "Footprint" "LED_THT:LED_D5.0mm-4_RGB" (at 261.62 152.4 0)
+    (property "Footprint" "LED_THT:LED_D5.0mm-4_RGB_Staggered_Pins" (at 261.62 152.4 0)
       (effects (font (size 1.27 1.27)) hide)
     )
@@
       (effects (font (size 1.27 1.27)))
     )
-    (property "Footprint" "LED_THT:LED_D5.0mm-4_RGB" (at 261.62 106.68 0)
+    (property "Footprint" "LED_THT:LED_D5.0mm-4_RGB_Staggered_Pins" (at 261.62 106.68 0)
       (effects (font (size 1.27 1.27)) hide)
     )
@@
     )
   )
+  (symbol (lib_id "Device:R") (at 55.88 72.39 0) (unit 1)
+    (in_bom yes) (on_board yes) (dnp no)
+    (property "Reference" "R2" (at 58.42 71.12 0)
+      (effects (font (size 1.27 1.27)) (justify left))
+    )
+    (property "Value" "11k" (at 58.42 73.66 0)
+      (effects (font (size 1.27 1.27)) (justify left))
+    )
+    (property "Footprint" "Resistor_SMD:R_0603_1608Metric" (at 54.102 72.39 90)
+      (effects (font (size 1.27 1.27)) hide)
+    )
+    (property "Datasheet" "~" (at 55.88 72.39 0)
+      (effects (font (size 1.27 1.27)) hide)
+    )
+    (pin "1")
+    (pin "2")
+    (instances
+      (project "cocoro"
+        (path "/d9dd42f0-aa5c-442e-a67c-269b1cf4745b/97ea76ca-9415-4083-9485-343aeb93230e"
+          (reference "R2") (unit 1)
+        )
+      )
+    )
+  )
   (symbol (lib_id "Device:LED_RKGB") (at 232.41 105.41 0) (mirror y) (unit 1)
     (in_bom yes) (on_board yes) (dnp no)
@@
       (effects (font (size 1.27 1.27)))
     )
-    (property "Footprint" "LED_THT:LED_D5.0mm-4_RGB" (at 232.41 106.68 0)
+    (property "Footprint" "LED_THT:LED_D5.0mm-4_RGB_Staggered_Pins" (at 232.41 106.68 0)
       (effects (font (size 1.27 1.27)) hide)
     )
@@
         )
         (path "/d9dd42f0-aa5c-442e-a67c-269b1cf4745b/97ea76ca-9415-4083-9485-343aeb93230e"
-          (reference "U2") (unit 1)
+          (reference "U3") (unit 1)
         )
       )
@@
   (symbol (lib_id "power:GND") (at 21.59 55.88 0) (unit 1)
     (in_bom yes) (on_board yes) (dnp no) (fields_autoplaced)
-    (property "Reference" "#PWR08" (at 21.59 62.23 0)
+    (property "Reference" "#PWR011" (at 21.59 62.23 0)
       (effects (font (size 1.27 1.27)) hide)
     )
@@
       (project "cocoro"
         (path "/d9dd42f0-aa5c-442e-a67c-269b1cf4745b/97ea76ca-9415-4083-9485-343aeb93230e"
-          (reference "#PWR08") (unit 1)
+          (reference "#PWR011") (unit 1)
         )
       )
@@
       (effects (font (size 1.27 1.27)))
     )
-    (property "Footprint" "LED_THT:LED_D5.0mm-4_RGB" (at 199.39 129.54 0)
+    (property "Footprint" "LED_THT:LED_D5.0mm-4_RGB_Staggered_Pins" (at 199.39 129.54 0)
       (effects (font (size 1.27 1.27)) hide)
     )
@@
       (effects (font (size 1.27 1.27)))
     )
-    (property "Footprint" "LED_THT:LED_D5.0mm-4_RGB" (at 199.39 83.82 0)
+    (property "Footprint" "LED_THT:LED_D5.0mm-4_RGB_Staggered_Pins" (at 199.39 83.82 0)
       (effects (font (size 1.27 1.27)) hide)
     )
@@
     )
   )
+  (symbol (lib_id "power:GND") (at 55.88 76.2 0) (unit 1)
+    (in_bom yes) (on_board yes) (dnp no)
+    (property "Reference" "#PWR06" (at 55.88 82.55 0)
+      (effects (font (size 1.27 1.27)) hide)
+    )
+    (property "Value" "GND" (at 55.88 81.28 0)
+      (effects (font (size 1.27 1.27)))
+    )
+    (property "Footprint" "" (at 55.88 76.2 0)
+      (effects (font (size 1.27 1.27)) hide)
+    )
+    (property "Datasheet" "" (at 55.88 76.2 0)
+      (effects (font (size 1.27 1.27)) hide)
+    )
+    (pin "1")
+    (instances
+      (project "cocoro"
+        (path "/d9dd42f0-aa5c-442e-a67c-269b1cf4745b"
+          (reference "#PWR06") (unit 1)
+        )
+        (path "/d9dd42f0-aa5c-442e-a67c-269b1cf4745b/97ea76ca-9415-4083-9485-343aeb93230e"
+          (reference "#PWR013") (unit 1)
+        )
+      )
+    )
+  )
   (symbol (lib_id "Device:LED_RKGB") (at 170.18 105.41 0) (mirror y) (unit 1)
     (in_bom yes) (on_board yes) (dnp no)
@@
       (effects (font (size 1.27 1.27)))
     )
-    (property "Footprint" "LED_THT:LED_D5.0mm-4_RGB" (at 170.18 106.68 0)
+    (property "Footprint" "LED_THT:LED_D5.0mm-4_RGB_Staggered_Pins" (at 170.18 106.68 0)
       (effects (font (size 1.27 1.27)) hide)
     )
@@
       (effects (font (size 1.27 1.27)))
     )
-    (property "Footprint" "LED_THT:LED_D5.0mm-4_RGB" (at 261.62 83.82 0)
+    (property "Footprint" "LED_THT:LED_D5.0mm-4_RGB_Staggered_Pins" (at 261.62 83.82 0)
       (effects (font (size 1.27 1.27)) hide)
     )
@@
       (effects (font (size 1.27 1.27)))
     )
-    (property "Footprint" "LED_THT:LED_D5.0mm-4_RGB" (at 261.62 129.54 0)
+    (property "Footprint" "LED_THT:LED_D5.0mm-4_RGB_Staggered_Pins" (at 261.62 129.54 0)
       (effects (font (size 1.27 1.27)) hide)
     )
@@
       (effects (font (size 1.27 1.27)))
     )
-    (property "Footprint" "LED_THT:LED_D5.0mm-4_RGB" (at 232.41 83.82 0)
+    (property "Footprint" "LED_THT:LED_D5.0mm-4_RGB_Staggered_Pins" (at 232.41 83.82 0)
       (effects (font (size 1.27 1.27)) hide)
     )
@@
       (effects (font (size 1.27 1.27)))
     )
-    (property "Footprint" "LED_THT:LED_D5.0mm-4_RGB" (at 199.39 106.68 0)
+    (property "Footprint" "LED_THT:LED_D5.0mm-4_RGB_Staggered_Pins" (at 199.39 106.68 0)
       (effects (font (size 1.27 1.27)) hide)
     )
@@
       (effects (font (size 1.27 1.27)))
     )
-    (property "Footprint" "LED_THT:LED_D5.0mm-4_RGB" (at 232.41 152.4 0)
+    (property "Footprint" "LED_THT:LED_D5.0mm-4_RGB_Staggered_Pins" (at 232.41 152.4 0)
       (effects (font (size 1.27 1.27)) hide)
     )
@@
       (effects (font (size 1.27 1.27)))
     )
-    (property "Footprint" "LED_THT:LED_D5.0mm-4_RGB" (at 232.41 129.54 0)
+    (property "Footprint" "LED_THT:LED_D5.0mm-4_RGB_Staggered_Pins" (at 232.41 129.54 0)
       (effects (font (size 1.27 1.27)) hide)
     )
@@
       (effects (font (size 1.27 1.27)))
     )
-    (property "Footprint" "LED_THT:LED_D5.0mm-4_RGB" (at 170.18 152.4 0)
+    (property "Footprint" "LED_THT:LED_D5.0mm-4_RGB_Staggered_Pins" (at 170.18 152.4 0)
       (effects (font (size 1.27 1.27)) hide)
     )
@@
       (effects (font (size 1.27 1.27)))
     )
-    (property "Footprint" "LED_THT:LED_D5.0mm-4_RGB" (at 170.18 129.54 0)
+    (property "Footprint" "LED_THT:LED_D5.0mm-4_RGB_Staggered_Pins" (at 170.18 129.54 0)
       (effects (font (size 1.27 1.27)) hide)
     )
@@
   (symbol (lib_id "Device:C") (at 21.59 52.07 0) (unit 1)
     (in_bom yes) (on_board yes) (dnp no) (fields_autoplaced)
-    (property "Reference" "C5" (at 25.4 50.8 0)
+    (property "Reference" "C9" (at 25.4 50.8 0)
       (effects (font (size 1.27 1.27)) (justify left))
     )
@@
       (project "cocoro"
         (path "/d9dd42f0-aa5c-442e-a67c-269b1cf4745b/97ea76ca-9415-4083-9485-343aeb93230e"
-          (reference "C5") (unit 1)
+          (reference "C9") (unit 1)
         )
       )
@@
       (effects (font (size 1.27 1.27)))
     )
-    (property "Footprint" "LED_THT:LED_D5.0mm-4_RGB" (at 170.18 83.82 0)
+    (property "Footprint" "LED_THT:LED_D5.0mm-4_RGB_Staggered_Pins" (at 170.18 83.82 0)
       (effects (font (size 1.27 1.27)) hide)
     )
@@
       (effects (font (size 1.27 1.27)))
     )
-    (property "Footprint" "LED_THT:LED_D5.0mm-4_RGB" (at 199.39 152.4 0)
-      (effects (font (size 1.27 1.27)) hide)
-    )
+    (property "Footprint" "LED_THT:LED_D5.0mm-4_RGB_Staggered_Pins" (at 199.39 152.4 0)
+      (effects (font (size 1.27 1.27)) hide)
+    )

Commit message: cocoro: Board touchups and decoupling caps
Performed minor touchup to reduce the size of ground islands. Added
some extra vias and decoupling caps for the power MOSFETs, since
it is recommended to add some extra capacitance to the voltage line
according to the LED1642 datasheet.
Parts:
- added C10, C11, C12: TBD, Capacitor_SMD:C_0805_2012Metric, symbol Device:C
Connections:
- net 5V: now also C10.1, C11.1, C12.1
- net GND: now also C10.2, C11.2, C12.2
Changed lines of the file:
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@@
 (kicad_sch (version 20230121) (generator eeschema)
   (paper "A4")
+  (junction (at 162.56 29.21) (diameter 0) (color 0 0 0 0)
+  )
   (junction (at 223.52 29.21) (diameter 0) (color 0 0 0 0)
   )
+  (junction (at 172.72 29.21) (diameter 0) (color 0 0 0 0)
+  )
   (junction (at 200.66 29.21) (diameter 0) (color 0 0 0 0)
   )
+  (junction (at 182.88 29.21) (diameter 0) (color 0 0 0 0)
+  )
   (wire (pts (xy 50.8 44.45) (xy 60.96 44.45))
     (stroke (width 0) (type default))
@@
     (stroke (width 0) (type default))
   )
+  (wire (pts (xy 172.72 29.21) (xy 182.88 29.21))
+    (stroke (width 0) (type default))
+  )
   (wire (pts (xy 59.69 54.61) (xy 60.96 54.61))
     (stroke (width 0) (type default))
@@
     (stroke (width 0) (type default))
   )
+  (wire (pts (xy 162.56 29.21) (xy 162.56 31.75))
+    (stroke (width 0) (type default))
+  )
   (wire (pts (xy 91.44 59.69) (xy 100.33 59.69))
     (stroke (width 0) (type default))
   )
+  (wire (pts (xy 172.72 29.21) (xy 172.72 31.75))
+    (stroke (width 0) (type default))
+  )
   (wire (pts (xy 223.52 30.48) (xy 223.52 29.21))
     (stroke (width 0) (type default))
@@
     (stroke (width 0) (type default))
   )
+  (wire (pts (xy 182.88 29.21) (xy 200.66 29.21))
+    (stroke (width 0) (type default))
+  )
+  (wire (pts (xy 162.56 29.21) (xy 172.72 29.21))
+    (stroke (width 0) (type default))
+  )
   (wire (pts (xy 91.44 54.61) (xy 100.33 54.61))
     (stroke (width 0) (type default))
@@
     (stroke (width 0) (type default))
   )
-  (wire (pts (xy 195.58 29.21) (xy 200.66 29.21))
+  (wire (pts (xy 158.75 29.21) (xy 162.56 29.21))
     (stroke (width 0) (type default))
   )
@@
   )
   (wire (pts (xy 223.52 29.21) (xy 246.38 29.21))
+    (stroke (width 0) (type default))
+  )
+  (wire (pts (xy 182.88 31.75) (xy 182.88 29.21))
     (stroke (width 0) (type default))
   )
@@
     )
   )
-  (global_label "5V" (shape input) (at 195.58 29.21 180) (fields_autoplaced)
-    (effects (font (size 1.27 1.27)) (justify right))
-    (property "Intersheetrefs" "${INTERSHEET_REFS}" (at 190.3761 29.21 0)
+  (global_label "5V" (shape input) (at 158.75 29.21 180) (fields_autoplaced)
+    (effects (font (size 1.27 1.27)) (justify right))
+    (property "Intersheetrefs" "${INTERSHEET_REFS}" (at 153.5461 29.21 0)
       (effects (font (size 1.27 1.27)) (justify right) hide)
     )
@@
         (path "/d9dd42f0-aa5c-442e-a67c-269b1cf4745b/97ea76ca-9415-4083-9485-343aeb93230e"
           (reference "D16") (unit 1)
+        )
+      )
+    )
+  )
+  (symbol (lib_id "power:GND") (at 172.72 39.37 0) (unit 1)
+    (in_bom yes) (on_board yes) (dnp no)
+    (property "Reference" "#PWR06" (at 172.72 45.72 0)
+      (effects (font (size 1.27 1.27)) hide)
+    )
+    (property "Value" "GND" (at 172.72 44.45 0)
+      (effects (font (size 1.27 1.27)))
+    )
+    (property "Footprint" "" (at 172.72 39.37 0)
+      (effects (font (size 1.27 1.27)) hide)
+    )
+    (property "Datasheet" "" (at 172.72 39.37 0)
+      (effects (font (size 1.27 1.27)) hide)
+    )
+    (pin "1")
+    (instances
+      (project "cocoro"
+        (path "/d9dd42f0-aa5c-442e-a67c-269b1cf4745b"
+          (reference "#PWR06") (unit 1)
+        )
+        (path "/d9dd42f0-aa5c-442e-a67c-269b1cf4745b/97ea76ca-9415-4083-9485-343aeb93230e"
+          (reference "#PWR016") (unit 1)
         )
       )
@@
     )
   )
+  (symbol (lib_id "Device:C") (at 182.88 35.56 0) (unit 1)
+    (in_bom yes) (on_board yes) (dnp no) (fields_autoplaced)
+    (property "Reference" "C10" (at 186.69 34.29 0)
+      (effects (font (size 1.27 1.27)) (justify left))
+    )
+    (property "Value" "TBD" (at 186.69 36.83 0)
+      (effects (font (size 1.27 1.27)) (justify left))
+    )
+    (property "Footprint" "Capacitor_SMD:C_0805_2012Metric" (at 183.8452 39.37 0)
+      (effects (font (size 1.27 1.27)) hide)
+    )
+    (property "Datasheet" "~" (at 182.88 35.56 0)
+      (effects (font (size 1.27 1.27)) hide)
+    )
+    (pin "1")
+    (pin "2")
+    (instances
+      (project "cocoro"
+        (path "/d9dd42f0-aa5c-442e-a67c-269b1cf4745b/97ea76ca-9415-4083-9485-343aeb93230e"
+          (reference "C10") (unit 1)
+        )
+      )
+    )
+  )
   (symbol (lib_id "Device:LED_RKGB") (at 199.39 128.27 0) (mirror y) (unit 1)
     (in_bom yes) (on_board yes) (dnp no)
@@
     )
   )
+  (symbol (lib_id "Device:C") (at 172.72 35.56 0) (unit 1)
+    (in_bom yes) (on_board yes) (dnp no) (fields_autoplaced)
+    (property "Reference" "C11" (at 176.53 34.29 0)
+      (effects (font (size 1.27 1.27)) (justify left))
+    )
+    (property "Value" "TBD" (at 176.53 36.83 0)
+      (effects (font (size 1.27 1.27)) (justify left))
+    )
+    (property "Footprint" "Capacitor_SMD:C_0805_2012Metric" (at 173.6852 39.37 0)
+      (effects (font (size 1.27 1.27)) hide)
+    )
+    (property "Datasheet" "~" (at 172.72 35.56 0)
+      (effects (font (size 1.27 1.27)) hide)
+    )
+    (pin "1")
+    (pin "2")
+    (instances
+      (project "cocoro"
+        (path "/d9dd42f0-aa5c-442e-a67c-269b1cf4745b/97ea76ca-9415-4083-9485-343aeb93230e"
+          (reference "C11") (unit 1)
+        )
+      )
+    )
+  )
+  (symbol (lib_id "power:GND") (at 182.88 39.37 0) (unit 1)
+    (in_bom yes) (on_board yes) (dnp no)
+    (property "Reference" "#PWR06" (at 182.88 45.72 0)
+      (effects (font (size 1.27 1.27)) hide)
+    )
+    (property "Value" "GND" (at 182.88 44.45 0)
+      (effects (font (size 1.27 1.27)))
+    )
+    (property "Footprint" "" (at 182.88 39.37 0)
+      (effects (font (size 1.27 1.27)) hide)
+    )
+    (property "Datasheet" "" (at 182.88 39.37 0)
+      (effects (font (size 1.27 1.27)) hide)
+    )
+    (pin "1")
+    (instances
+      (project "cocoro"
+        (path "/d9dd42f0-aa5c-442e-a67c-269b1cf4745b"
+          (reference "#PWR06") (unit 1)
+        )
+        (path "/d9dd42f0-aa5c-442e-a67c-269b1cf4745b/97ea76ca-9415-4083-9485-343aeb93230e"
+          (reference "#PWR015") (unit 1)
+        )
+      )
+    )
+  )
   (symbol (lib_id "power:GND") (at 55.88 76.2 0) (unit 1)
     (in_bom yes) (on_board yes) (dnp no)
@@
         (path "/d9dd42f0-aa5c-442e-a67c-269b1cf4745b/97ea76ca-9415-4083-9485-343aeb93230e"
           (reference "D9") (unit 1)
+        )
+      )
+    )
+  )
+  (symbol (lib_id "power:GND") (at 162.56 39.37 0) (unit 1)
+    (in_bom yes) (on_board yes) (dnp no)
+    (property "Reference" "#PWR06" (at 162.56 45.72 0)
+      (effects (font (size 1.27 1.27)) hide)
+    )
+    (property "Value" "GND" (at 162.56 44.45 0)
+      (effects (font (size 1.27 1.27)))
+    )
+    (property "Footprint" "" (at 162.56 39.37 0)
+      (effects (font (size 1.27 1.27)) hide)
+    )
+    (property "Datasheet" "" (at 162.56 39.37 0)
+      (effects (font (size 1.27 1.27)) hide)
+    )
+    (pin "1")
+    (instances
+      (project "cocoro"
+        (path "/d9dd42f0-aa5c-442e-a67c-269b1cf4745b"
+          (reference "#PWR06") (unit 1)
+        )
+        (path "/d9dd42f0-aa5c-442e-a67c-269b1cf4745b/97ea76ca-9415-4083-9485-343aeb93230e"
+          (reference "#PWR017") (unit 1)
         )
       )
@@
         )
       )
+    )
+  )
+  (symbol (lib_id "Device:C") (at 162.56 35.56 0) (unit 1)
+    (in_bom yes) (on_board yes) (dnp no) (fields_autoplaced)
+    (property "Reference" "C12" (at 166.37 34.29 0)
+      (effects (font (size 1.27 1.27)) (justify left))
+    )
+    (property "Value" "TBD" (at 166.37 36.83 0)
+      (effects (font (size 1.27 1.27)) (justify left))
+    )
+    (property "Footprint" "Capacitor_SMD:C_0805_2012Metric" (at 163.5252 39.37 0)
+      (effects (font (size 1.27 1.27)) hide)
+    )
+    (property "Datasheet" "~" (at 162.56 35.56 0)
+      (effects (font (size 1.27 1.27)) hide)
+    )
+    (pin "1")
+    (pin "2")
+    (instances
+      (project "cocoro"
+        (path "/d9dd42f0-aa5c-442e-a67c-269b1cf4745b/97ea76ca-9415-4083-9485-343aeb93230e"
+          (reference "C12") (unit 1)
+        )
+      )

Commit message: Housekeeping, deleted extra-crappy projects, add CI
Deleted a bunch of half-finished projects that won't be getting
attention anytime soon:

* filscrete-8bp: Making a good quality filter for the VHF band will be
  much harder than expected and won't be pursued for the time being.
* ev1496: Much more investigation needs to be done on the intrinsic
  characteristics of the MC1496 IC before being able to develop an
  evaluation board.
* sam: Very ambitious project, will start first with smaller ones.

Library symbols for these projects have been kept since they mave prove
useful in the future.

Front matter has been added to the remaining project. It is planned to
automatically create a portfolio website for this repo with balba:

https://gitlab.com/zoftko/balba

And a standard front matter will be needed for that.

Finally, a basic CI with pre-commit has been added to improve code
quality. In the future it should also perform spell checks.
Other:
- title: (none) -> RGB LED Array controlling circuitry
Changed lines of the file:
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@@
 (kicad_sch (version 20230121) (generator eeschema)
   (paper "A4")
+  (title_block
+    (title "RGB LED Array controlling circuitry")
+  )
   (junction (at 162.56 29.21) (diameter 0) (color 0 0 0 0)
   )
