File: cocoro/ledc.kicad_sch (KiCad schematic)
At the start: 25 parts, among them Q1 FDN340P, Q2 FDN340P, Q3 FDN340P, U1 LED1642GWTTR

Commit message: Update cocoro to kicad v8, add notes
Board was originally designed in Kicad 7, Kicad 8 is now out and
opening boards from older versions automatically converts them so might
as well do it now.

There is also an error on the board, it has been noted in its README.
Parts:
- renumbered D2 to D1, D11 to D10, D12 to D11, D13 to D12, D14 to D13, D15 to D14, D16 to D15, D17 to D16, D3 to D2, D4 to D3, D5 to D4, D6 to D5, D7 to D6, D8 to D7, D9 to D8, D10 to D9, U1 to U3
