File: zcd393/zcd393.kicad_pcb (KiCad board)
At the start: 4 copper layers, 25 x 38 mm, 18 parts, among them J1 Screw_Terminal_01x02, J2 Conn_01x05_Pin, U1 LM393

Commit message: Fix diode footprint
Parts:
- D1: footprint Diode_SMD:D_SOD-323 -> Diode_SMD:D_SOD-123
- moved D1 0.90 mm to (161.0, 98.5)
Changed lines of the file:
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@@
     )
   )
-  (footprint "Diode_SMD:D_SOD-323" (layer "F.Cu")
-    (at 160.25 98)
-    (descr "SOD-323")
-    (tags "SOD-323")
+  (footprint "Diode_SMD:D_SOD-123" (layer "F.Cu")
+    (at 161 98.5)
+    (descr "SOD-123")
+    (tags "SOD-123")
     (property "Sheetfile" "zcd393.kicad_sch")
     (property "Sheetname" "")
@@
     (property "ki_keywords" "diode Schottky")
     (attr smd)
-    (fp_text reference "D1" (at 2.625 0) (layer "F.SilkS")
-        (effects (font (size 1 1) (thickness 0.15)))
-    )
-    (fp_text value "1N5819WS" (at 0.1 1.9) (layer "F.Fab") hide
-        (effects (font (size 1 1) (thickness 0.15)))
-    )
-    (fp_line (start -1.61 -0.85) (end -1.61 0.85)
-      (stroke (width 0.12) (type solid)) (layer "F.SilkS"))
-    (fp_line (start -1.61 -0.85) (end 1.05 -0.85)
-      (stroke (width 0.12) (type solid)) (layer "F.SilkS"))
-    (fp_line (start -1.61 0.85) (end 1.05 0.85)
-      (stroke (width 0.12) (type solid)) (layer "F.SilkS"))
-    (fp_line (start -1.6 -0.95) (end -1.6 0.95)
-      (stroke (width 0.05) (type solid)) (layer "F.CrtYd"))
-    (fp_line (start -1.6 -0.95) (end 1.6 -0.95)
-      (stroke (width 0.05) (type solid)) (layer "F.CrtYd"))
-    (fp_line (start -1.6 0.95) (end 1.6 0.95)
-      (stroke (width 0.05) (type solid)) (layer "F.CrtYd"))
-    (fp_line (start 1.6 -0.95) (end 1.6 0.95)
-      (stroke (width 0.05) (type solid)) (layer "F.CrtYd"))
-    (fp_line (start -0.9 -0.7) (end 0.9 -0.7)
-      (stroke (width 0.1) (type solid)) (layer "F.Fab"))
-    (fp_line (start -0.9 0.7) (end -0.9 -0.7)
-      (stroke (width 0.1) (type solid)) (layer "F.Fab"))
-    (fp_line (start -0.3 -0.35) (end -0.3 0.35)
-      (stroke (width 0.1) (type solid)) (layer "F.Fab"))
-    (fp_line (start -0.3 0) (end -0.5 0)
-      (stroke (width 0.1) (type solid)) (layer "F.Fab"))
-    (fp_line (start -0.3 0) (end 0.2 -0.35)
-      (stroke (width 0.1) (type solid)) (layer "F.Fab"))
-    (fp_line (start 0.2 -0.35) (end 0.2 0.35)
-      (stroke (width 0.1) (type solid)) (layer "F.Fab"))
-    (fp_line (start 0.2 0) (end 0.45 0)
-      (stroke (width 0.1) (type solid)) (layer "F.Fab"))
-    (fp_line (start 0.2 0.35) (end -0.3 0)
-      (stroke (width 0.1) (type solid)) (layer "F.Fab"))
-    (fp_line (start 0.9 -0.7) (end 0.9 0.7)
-      (stroke (width 0.1) (type solid)) (layer "F.Fab"))
-    (fp_line (start 0.9 0.7) (end -0.9 0.7)
-      (stroke (width 0.1) (type solid)) (layer "F.Fab"))
-    (pad "1" smd roundrect (at -1.05 0) (size 0.6 0.45) (layers "F.Cu" "F.Paste" "F.Mask") (roundrect_rratio 0.25)
+    (fp_text reference "D1" (at 0 2) (layer "F.SilkS")
+        (effects (font (size 1 1) (thickness 0.15)))
+    )
+    (fp_text value "1N5819WS" (at 0 2.1) (layer "F.Fab") hide
+        (effects (font (size 1 1) (thickness 0.15)))
+    )
+    (fp_text user "${REFERENCE}" (at 0 -2) (layer "F.Fab")
+        (effects (font (size 1 1) (thickness 0.15)))
+    )
+    (fp_line (start -2.36 -1) (end -2.36 1)
+      (stroke (width 0.12) (type solid)) (layer "F.SilkS"))
+    (fp_line (start -2.36 -1) (end 1.65 -1)
+      (stroke (width 0.12) (type solid)) (layer "F.SilkS"))
+    (fp_line (start -2.36 1) (end 1.65 1)
+      (stroke (width 0.12) (type solid)) (layer "F.SilkS"))
+    (fp_line (start -2.35 -1.15) (end -2.35 1.15)
+      (stroke (width 0.05) (type solid)) (layer "F.CrtYd"))
+    (fp_line (start -2.35 -1.15) (end 2.35 -1.15)
+      (stroke (width 0.05) (type solid)) (layer "F.CrtYd"))
+    (fp_line (start 2.35 -1.15) (end 2.35 1.15)
+      (stroke (width 0.05) (type solid)) (layer "F.CrtYd"))
+    (fp_line (start 2.35 1.15) (end -2.35 1.15)
+      (stroke (width 0.05) (type solid)) (layer "F.CrtYd"))
+    (fp_line (start -1.4 -0.9) (end 1.4 -0.9)
+      (stroke (width 0.1) (type solid)) (layer "F.Fab"))
+    (fp_line (start -1.4 0.9) (end -1.4 -0.9)
+      (stroke (width 0.1) (type solid)) (layer "F.Fab"))
+    (fp_line (start -0.75 0) (end -0.35 0)
+      (stroke (width 0.1) (type solid)) (layer "F.Fab"))
+    (fp_line (start -0.35 0) (end -0.35 -0.55)
+      (stroke (width 0.1) (type solid)) (layer "F.Fab"))
+    (fp_line (start -0.35 0) (end -0.35 0.55)
+      (stroke (width 0.1) (type solid)) (layer "F.Fab"))
+    (fp_line (start -0.35 0) (end 0.25 -0.4)
+      (stroke (width 0.1) (type solid)) (layer "F.Fab"))
+    (fp_line (start 0.25 -0.4) (end 0.25 0.4)
+      (stroke (width 0.1) (type solid)) (layer "F.Fab"))
+    (fp_line (start 0.25 0) (end 0.75 0)
+      (stroke (width 0.1) (type solid)) (layer "F.Fab"))
+    (fp_line (start 0.25 0.4) (end -0.35 0)
+      (stroke (width 0.1) (type solid)) (layer "F.Fab"))
+    (fp_line (start 1.4 -0.9) (end 1.4 0.9)
+      (stroke (width 0.1) (type solid)) (layer "F.Fab"))
+    (fp_line (start 1.4 0.9) (end -1.4 0.9)
+      (stroke (width 0.1) (type solid)) (layer "F.Fab"))
+    (pad "1" smd roundrect (at -1.65 0) (size 0.9 1.2) (layers "F.Cu" "F.Paste" "F.Mask") (roundrect_rratio 0.25)
       (net 5 "/ACATT") (pinfunction "K") (pintype "passive"))
-    (pad "2" smd roundrect (at 1.05 0) (size 0.6 0.45) (layers "F.Cu" "F.Paste" "F.Mask") (roundrect_rratio 0.25)
+    (pad "2" smd roundrect (at 1.65 0) (size 0.9 1.2) (layers "F.Cu" "F.Paste" "F.Mask") (roundrect_rratio 0.25)
       (net 2 "GND") (pinfunction "A") (pintype "passive"))
-    (model "${KICAD6_3DMODEL_DIR}/Diode_SMD.3dshapes/D_SOD-323.wrl"
+    (model "${KICAD6_3DMODEL_DIR}/Diode_SMD.3dshapes/D_SOD-123.wrl"
       (offset (xyz 0 0 0))
       (scale (xyz 1 1 1))
@@
     (property "ki_keywords" "screw terminal")
     (attr through_hole)
-    (fp_text reference "J1" (at 1 -3.5 unlocked) (layer "F.SilkS")
+    (fp_text reference "J1" (at -9.2 -0.75 unlocked) (layer "F.SilkS")
         (effects (font (size 1 1) (thickness 0.1)))
     )
@@
     (effects (font (size 1 1) (thickness 0.15)) (justify left bottom))
   )
-  (gr_text "ZCD393" (at 163 101) (layer "F.SilkS")
+  (gr_text "ZCD393" (at 163.5 101.5) (layer "F.SilkS")
     (effects (font (size 1.5 1.5) (thickness 0.15)) (justify left bottom))
   )
@@
   (via (at 165 85) (size 1) (drill 0.6) (layers "F.Cu" "B.Cu") (free) (net 2))
   (via (at 152 98) (size 1) (drill 0.6) (layers "F.Cu" "B.Cu") (free) (net 2))
-  (via (at 164.75 98) (size 1) (drill 0.6) (layers "F.Cu" "B.Cu") (free) (net 2))
+  (via (at 164.75 98.5) (size 1) (drill 0.6) (layers "F.Cu" "B.Cu") (free) (net 2))
   (via (at 154 85) (size 1) (drill 0.6) (layers "F.Cu" "B.Cu") (free) (net 2))
   (segment (start 156.7 99.825) (end 156.7 104.75) (width 0.4) (layer "F.Cu") (net 3))
@@
   (segment (start 159.425 96) (end 158.5 96) (width 0.4) (layer "F.Cu") (net 5))
   (segment (start 158.5 96) (end 157.625 96.875) (width 0.4) (layer "F.Cu") (net 5))
-  (segment (start 158.25 98) (end 157.625 97.375) (width 0.4) (layer "F.Cu") (net 5))
+  (segment (start 159.35 98.5) (end 158.75 98.5) (width 0.4) (layer "F.Cu") (net 5))
   (segment (start 156.85 96) (end 156.675 95.825) (width 0.4) (layer "F.Cu") (net 5))
   (segment (start 156.7 95.85) (end 156.675 95.825) (width 0.4) (layer "F.Cu") (net 5))
   (segment (start 157.625 96.875) (end 157.5 97) (width 0.4) (layer "F.Cu") (net 5))
+  (segment (start 157.625 97.375) (end 157.625 96.875) (width 0.4) (layer "F.Cu") (net 5))
+  (segment (start 158.75 98.5) (end 157.625 97.375) (width 0.4) (layer "F.Cu") (net 5))
   (segment (start 156.7 97) (end 156.7 95.85) (width 0.4) (layer "F.Cu") (net 5))
-  (segment (start 157.625 97.375) (end 157.625 96.875) (width 0.4) (layer "F.Cu") (net 5))
   (segment (start 156.7 98.175) (end 156.7 97) (width 0.4) (layer "F.Cu") (net 5))
-  (segment (start 159.2 98) (end 158.25 98) (width 0.4) (layer "F.Cu") (net 5))
   (segment (start 157.5 97) (end 156.7 97) (width 0.4) (layer "F.Cu") (net 5))
   (segment (start 156.675 94.175) (end 156.675 93) (width 0.4) (layer "F.Cu") (net 6))
