File: zcd393/zcd393.kicad_sch (KiCad schematic)
At the start: 18 parts, among them J1 Screw_Terminal_01x02, J2 Conn_01x05_Pin, U1 LM393

Commit message: Fix diode footprint
Parts:
- D1: footprint Diode_SMD:D_SOD-323 -> Diode_SMD:D_SOD-123
Changed lines of the file:
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@@
       (effects (font (size 1.27 1.27)) (justify left))
     )
-    (property "Footprint" "Diode_SMD:D_SOD-323" (at 128.905 105.41 0)
+    (property "Footprint" "Diode_SMD:D_SOD-123" (at 128.905 105.41 0)
       (effects (font (size 1.27 1.27)) hide)
     )
