File: pcroast/pcroast.kicad_pcb (KiCad board)
At the start: 4 copper layers, 99.6 x 70 mm, 45 parts, among them J1 Screw_Terminal_01x02, J2 Barrel_Jack_Switch, J3 Screw_Terminal_01x02, J4 Conn_01x08_Pin, J5 Screw_Terminal_01x02, J6 Conn_01x02_Pin, J7 Conn_01x03_Pin, Q1 IRLML2502, Q2 FDN340P, Q3 IRLML2502, Q4 IRLML2502, Q5 IRLML2502, SW1 SW_Push, SW2 SW_Push, SW3 SW_Push, U1 MAX6675, U2 LM393, U3 PicoW

Commit message: Fix supply voltage for ZCD
It should be fed from 3.3V instead of 5V, as the RP2040 gpio pins should
not be exposed to 5V.
Parts:
- moved J6 1.03 mm to (164.0, 102.8)
Connections:
- C5 pad 1: +5V -> +3.3V
- R10 pad 2: +5V -> +3.3V
- R5 pad 1: +5V -> +3.3V
- R6 pad 1: +5V -> +3.3V
- U2 pad 8: +5V -> +3.3V
Routing:
- net +3.3V: track 94.0 -> 190.4 mm, vias 1 -> 4
- net +5V: track 290.0 -> 215.3 mm, vias 2 -> 0
- net /TX: track 7.12 -> 6.09 mm
- net /RX: track 7.12 -> 6.09 mm

Commit message: fix: ground T- termocouple probe
Parts:
- R7: value 220k -> 15k
Connections:
- J1 pad 1: /T- -> GND
- U1 pad 2: /T- -> GND
Routing:
- net /T-: track 11.9 -> 0.00 mm
- net GND: track 0.00 -> 1.50 mm
- net +5V: track 215.3 -> 214.5 mm
