File: pcroast/pcroast.kicad_sch (KiCad schematic)
At the start: 45 parts, among them J1 Screw_Terminal_01x02, J2 Barrel_Jack_Switch, J3 Screw_Terminal_01x02, J4 Conn_01x08_Pin, J5 Screw_Terminal_01x02, J6 Conn_01x02_Pin, J7 Conn_01x03_Pin, Q1 IRLML2502, Q2 FDN340P, Q3 IRLML2502, Q4 IRLML2502, Q5 IRLML2502, SW1 SW_Push, SW2 SW_Push, SW3 SW_Push, U1 MAX6675, U2 LM393, U3 PicoW

Commit message: Fix supply voltage for ZCD
It should be fed from 3.3V instead of 5V, as the RP2040 gpio pins should
not be exposed to 5V.
Connections:
- net +3.3V: now also C5.1, R10.2, R5.1, R6.1, U2.8 (V+)
- net +5V: no longer C5.1, R10.2, R5.1, R6.1, U2.8 (V+)
Changed lines of the file:
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@@
+    )
+  )
+  (symbol (lib_id "power:+3.3V") (at 93.98 128.27 0) (unit 1)
+    (in_bom yes) (on_board yes) (dnp no) (fields_autoplaced)
+    (property "Reference" "#PWR020" (at 93.98 132.08 0)
+      (effects (font (size 1.27 1.27)) hide)
+    )
+    (property "Value" "+3.3V" (at 93.98 123.19 0)
+      (effects (font (size 1.27 1.27)))
+    )
+    (property "Footprint" "" (at 93.98 128.27 0)
+      (effects (font (size 1.27 1.27)) hide)
+    )
+    (property "Datasheet" "" (at 93.98 128.27 0)
+      (effects (font (size 1.27 1.27)) hide)
+    )
+    (pin "1")
+    (instances
+      (project "pcroast"
+        (path "/3b27695c-a5de-4be8-932a-237690def1bd"
+          (reference "#PWR020") (unit 1)
+        )
+      )
     )
   )
@@
         (path "/3b27695c-a5de-4be8-932a-237690def1bd"
           (reference "Q2") (unit 1)
-        )
-      )
-    )
-  )
-  (symbol (lib_id "power:+5V") (at 93.98 128.27 0) (unit 1)
-    (in_bom yes) (on_board yes) (dnp no) (fields_autoplaced)
-    (property "Reference" "#PWR012" (at 93.98 132.08 0)
-      (effects (font (size 1.27 1.27)) hide)
-    )
-    (property "Value" "+5V" (at 93.98 123.19 0)
-      (effects (font (size 1.27 1.27)))
-    )
-    (property "Footprint" "" (at 93.98 128.27 0)
-      (effects (font (size 1.27 1.27)) hide)
-    )
-    (property "Datasheet" "" (at 93.98 128.27 0)
-      (effects (font (size 1.27 1.27)) hide)
-    )
-    (pin "1")
-    (instances
-      (project "pcroast"
-        (path "/3b27695c-a5de-4be8-932a-237690def1bd"
-          (reference "#PWR012") (unit 1)
         )
       )
@@
     )
   )
+  (symbol (lib_id "power:+3.3V") (at 121.92 152.4 0) (unit 1)
+    (in_bom yes) (on_board yes) (dnp no) (fields_autoplaced)
+    (property "Reference" "#PWR012" (at 121.92 156.21 0)
+      (effects (font (size 1.27 1.27)) hide)
+    )
+    (property "Value" "+3.3V" (at 121.92 147.32 0)
+      (effects (font (size 1.27 1.27)))
+    )
+    (property "Footprint" "" (at 121.92 152.4 0)
+      (effects (font (size 1.27 1.27)) hide)
+    )
+    (property "Datasheet" "" (at 121.92 152.4 0)
+      (effects (font (size 1.27 1.27)) hide)
+    )
+    (pin "1")
+    (instances
+      (project "pcroast"
+        (path "/3b27695c-a5de-4be8-932a-237690def1bd"
+          (reference "#PWR012") (unit 1)
+        )
+      )
+    )
+  )
   (symbol (lib_id "Device:R") (at 125.73 160.02 0) (unit 1)
     (in_bom yes) (on_board yes) (dnp no)
@@
         )
       )
-    )
-  )
-  (symbol (lib_id "power:+5V") (at 121.92 152.4 0) (unit 1)
-    (in_bom yes) (on_board yes) (dnp no) (fields_autoplaced)
-    (property "Reference" "#PWR020" (at 121.92 156.21 0)
-      (effects (font (size 1.27 1.27)) hide)
-    )
-    (property "Value" "+5V" (at 121.92 147.32 0)
-      (effects (font (size 1.27 1.27)))
-    )
-    (property "Footprint" "" (at 121.92 152.4 0)
-      (effects (font (size 1.27 1.27)) hide)
-    )
-    (property "Datasheet" "" (at 121.92 152.4 0)
-      (effects (font (size 1.27 1.27)) hide)
-    )
-    (pin "1")
-    (instances
-      (project "pcroast"
-        (path "/3b27695c-a5de-4be8-932a-237690def1bd"
-          (reference "#PWR020") (unit 1)
-        )
-      )

Commit message: fix: ground T- termocouple probe
Parts:
- R7: value 220k -> 15k
Connections:
- net T- is gone; now on net GND: J1.1 (Pin_1), U1.2 (T-)
Changed lines of the file:
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@@
   (junction (at 26.67 90.17) (diameter 0) (color 0 0 0 0)
+  )
+  (junction (at 31.75 104.14) (diameter 0) (color 0 0 0 0)
   )
   (junction (at 96.52 172.72) (diameter 0) (color 0 0 0 0)
@@
     (stroke (width 0) (type default))
   )
+  (wire (pts (xy 31.75 104.14) (xy 35.56 104.14))
+    (stroke (width 0) (type default))
+  )
   (wire (pts (xy 104.14 87.63) (xy 113.03 87.63))
     (stroke (width 0) (type default))
@@
     (stroke (width 0) (type default))
   )
+  (wire (pts (xy 31.75 104.14) (xy 31.75 106.68))
+    (stroke (width 0) (type default))
+  )
   (wire (pts (xy 250.19 100.33) (xy 250.19 113.03))
     (stroke (width 0) (type default))
@@
     (stroke (width 0) (type default))
   )
-  (wire (pts (xy 21.59 104.14) (xy 35.56 104.14))
+  (wire (pts (xy 21.59 104.14) (xy 31.75 104.14))
     (stroke (width 0) (type default))
   )
@@
       (effects (font (size 1.27 1.27)) (justify left))
     )
-    (property "Value" "220k" (at 128.27 185.42 0)
+    (property "Value" "15k" (at 128.27 185.42 0)
       (effects (font (size 1.27 1.27)) (justify left))
     )
@@
         )
       )
+    )
+  )
+  (symbol (lib_name "GND_11") (lib_id "power:GND") (at 31.75 106.68 0) (unit 1)
+    (in_bom yes) (on_board yes) (dnp no) (fields_autoplaced)
+    (property "Reference" "#PWR036" (at 31.75 113.03 0)
+      (effects (font (size 1.27 1.27)) hide)
+    )
+    (property "Value" "GND" (at 31.75 111.76 0)
+      (effects (font (size 1.27 1.27)))
+    )
+    (property "Footprint" "" (at 31.75 106.68 0)
+      (effects (font (size 1.27 1.27)) hide)
+    )
+    (property "Datasheet" "" (at 31.75 106.68 0)
+      (effects (font (size 1.27 1.27)) hide)
+    )
+    (pin "1")
+    (instances
+      (project "pcroast"
+        (path "/3b27695c-a5de-4be8-932a-237690def1bd"
+          (reference "#PWR036") (unit 1)
+        )
+      )
